File: X2C_DC_SHIELD.sch (EAGLE design)
At the start: 59 parts, among them CON1 X2C_PINHD-4X14_SMD, IC1 MCP16251, IC2 MCP6004ST, IC3 7408, T1 DMG6602SVT, T2 DMG6602SVT

Commit message: Updated amplifier values
Parts:
- removed LED5, LED6, LED7, LED8: Green, KANDO_KOZOS:LEDCHIPLED_0805_GREEN
- added LED1H, LED2H: Green, KANDO_KOZOS:LEDCHIPLED_0805_GREEN
- added R28, R29, R30: 680R, KANDO_KOZOS_V2:R-EU_SMDR0603_680R
- added R31: 2,2k, KANDO_KOZOS:R-EU_SMDR0603_2,2K
- added R32: 68k 1%, KANDO_KOZOS_V2:R-EU_SMDR0603_68K_1%
- C10, C5, C7, C8: value 2,2nF -> 22nF; device KANDO_KOZOS:C-EU-SMD_0603_2,2NF -> C_EU_Kando:C-EU-SMD_0603_22NF_16V
- C11: value 2,2nF -> 1uF; device KANDO_KOZOS:C-EU-SMD_0603_2,2NF -> KANDO_KOZOS_V2:C-EU-SMD_0603_1UF_10V
- C3: device C_EU_Kando:C-EU-SMD_0805_10UF_16V -> KANDO_KOZOS:C-EU-SMD_0805_10UF_16V
- C6: value 2,2nF -> 4,7uF; device KANDO_KOZOS:C-EU-SMD_0603_2,2NF -> C_EU_Kando:C-EU-SMD_0603_4,7UF_16V
- C9: value 100nF -> 1uF; device KANDO_KOZOS:C-EU-SMD_0603_100NF_50V -> C_EU_Kando:C-EU-SMD_0603_1UF_10V
- MOT1: device KANDO_KOZOS:DC_MOTOR_1 -> KANDO_KOZOS_V2:DC_MOTOR_1
- R1: value 330R -> 680R; device KANDO_KOZOS:4R-N330R -> KANDO_KOZOS_V2:R-EU_SMDR0603_680R
- R14, R15: value 330R -> 4,7k; device KANDO_KOZOS:R-EU_SMDR0603_330R -> R_EU:R-EU_SMDR0603_4,7K
- R16, R21, R22: value 22k 1% -> 68k 1%; device KANDO_KOZOS:R-EU_SMDR0603_22K_1% -> KANDO_KOZOS_V2:R-EU_SMDR0603_68K_1%
- R23, R24: value 2,2k -> 22k 1%; device KANDO_KOZOS:R-EU_SMDR0603_2,2K -> KANDO_KOZOS_V2:R-EU_SMDR0603_22K_1%
- R3: value 330R -> 680R; device KANDO_KOZOS:R-EU_SMDR0603_330R -> KANDO_KOZOS_V2:R-EU_SMDR0603_680R
- R4: value 2,2k -> 330k 1%; device KANDO_KOZOS:R-EU_SMDR0603_2,2K -> KANDO_KOZOS_V2:R-EU_SMDR0603_330K_1%
- R6: value 68k 1% -> 330k 1%; device KANDO_KOZOS:R-EU_SMDR0603_68K_1% -> KANDO_KOZOS_V2:R-EU_SMDR0603_330K_1%
- renumbered LED1 to LED3V3, LED2 to LED5V, LED3 to LED1L, LED4 to LED2L
Connections:
- removed net N$11: C6.2, IC2A.-IN, R12.2, R16.1
- net +3V3: now also MOT1.EMIT, R29.1, R30.1; no longer R14.2, R15.2
- net GND: now also C6.2, R1.1, R14.2, R15.2, R28.1; no longer MOT1.EMIT, R1A.2, R1B.2, R1C.2, R1D.2
- net IMOTOR: now also R32.2
- net N$10: now also R1.2; no longer R1A.1
- net N$13: now also LED1H.A, R30.2; no longer LED2L.C, R1B.1
- net N$14: now also LED2L.C, R28.2; no longer LED5.C, R1C.1
- net N$15: now also IC2A.-IN, R12.2, R16.1, R32.1; no longer LED6.C, R1D.1
- net N$16: now also C2.1, R31.2, R4.2; no longer LED8.A, R15.1
- net N$26: now also R31.1; no longer C2.1, R4.2
- net N$6: now also LED2H.A, R29.2; no longer LED7.A, R14.1
- net PWM1H: now also LED1H.C; no longer LED2L.A
- net PWM2H: now also LED2H.C; no longer LED6.A
- net PWM2L: now also LED2L.A; no longer LED5.A
- net QE_A: now also R14.1; no longer LED7.C
- net QE_B: now also R15.1; no longer LED8.C
Other:
- note added: "Generator Max Voltage: 5V (overdrive) 5-> 3.3/2 (zero shifted) Gain: 0.25"
- note removed: "Generator Max Voltage: 15V 15V->3.3/2 Gain: 0.11"
- moved on the sheet: C2, C6, R11, R12, R4
